File: FONA-Data-Logger-Board.brd (EAGLE design)
At the start: 50.8 x 50.8 mm, 46 parts

Commit message: Updated the Board and Schematic - Minor
Changed lines of the file:
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@@
 <text x="40.7924" y="12.3952" size="1.016" layer="21" font="vector" ratio="15">Power</text>
 <text x="55.4736" y="41.3004" size="1.27" layer="104" font="vector" ratio="15" rot="MR0">V5a</text>
-<text x="0.9652" y="24.4348" size="1.27" layer="25" font="vector" ratio="15">V4a</text>
+<text x="1.3208" y="24.4348" size="1.27" layer="25" font="vector" ratio="15">V4a</text>
 <text x="17.6022" y="1.8796" size="1.016" layer="25" font="vector" ratio="10" rot="R180">chip@mcclellands.org</text>
 <wire x1="38.9382" y1="26.3144" x2="38.9382" y2="25.2984" width="0.1016" layer="145"/>
